Commit message: *URDF changestatus increase mass for chassis to prevent fall in gazebo; also increased move_base velocities

File: movo_common/movo_description/urdf/movo_components/movo_base.urdf.xacro (robot description, xacro)
@@ -45,5 +45,5 @@
         <link name="base_chassis_link">
 			<inertial>
-				<mass value="44.2877" />
+				<mass value="95.2877" />
 				<origin xyz="-0.009506 -0.013039 0.032319" />
 				<inertia ixx="0.000165"  ixy="0" ixz="0"

Commit message: gazebo work pause

File: movo_common/movo_description/urdf/movo_components/movo_base.urdf.xacro (robot description, xacro)
@@ -45,5 +45,5 @@
         <link name="base_chassis_link">
 			<inertial>
-				<mass value="95.2877" />
+				<mass value="44.2877" />
 				<origin xyz="-0.009506 -0.013039 0.032319" />
 				<inertia ixx="0.000165"  ixy="0" ixz="0"
